File: BTIBR_ProjetoEletronico/BTIBR-PCB.kicad_pcb (KiCad board)
At the start: 2 copper layers, 200 x 77 mm, 78 parts, among them J1 Screw_Terminal_01x03, J10 Screw_Terminal_01x03, J11 Conn_01x03_Male, J12 Screw_Terminal_01x03, J13 Conn_01x09_Male, J14 Screw_Terminal_01x04, J15 Conn_01x07_Male, J16 Screw_Terminal_01x03, J2 Conn_01x04_Male, J3 Conn_01x09_Male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

Commit message: Correção do footprint do modulo pot digital
Routing:
- net Net-(C11-Pad1): track 22.6 -> 25.6 mm
- net Net-(C3-Pad1): track 23.4 -> 26.2 mm
- net Net-(C15-Pad1): track 23.5 -> 25.5 mm
- net +5V: track 373.7 -> 372.5 mm
- net Net-(J2-Pad3): track 9.93 -> 9.43 mm
- net Net-(J2-Pad2): track 9.93 -> 9.43 mm
- net Net-(J2-Pad1): track 9.93 -> 9.43 mm
- net Net-(J11-Pad3): track 9.93 -> 9.43 mm
- net Net-(J11-Pad2): track 9.93 -> 9.43 mm
- net Net-(J11-Pad1): track 9.93 -> 9.43 mm
